Commit message: all

File: RA605_710.SLDASM/robots/RA605_710.SLDASM.urdf (robot description, URDF)
Before this commit: robot RA605_710, 3 links, 2 joints
Links:
- link Link1: geometry collision mesh filename=package://RA605_710.SLDASM/meshes/Link1.STL; visual mesh filename=package://RA605_710.SLDASM/meshes/Link1.STL
- link Link2: geometry collision mesh filename=package://RA605_710.SLDASM/meshes/Link2.STL; visual mesh filename=package://RA605_710.SLDASM/meshes/Link2.STL
- link base_link: mass 39.9992146018366 -> 39.999; geometry collision mesh filename=package://RA605_710.SLDASM/meshes/base_link.STL; visual mesh filename=package://RA605_710.SLDASM/meshes/base_link.STL
Joints:
- joint j2: limit (none) -> lower=-3.1 upper=3.1 effort=0 velocity=0; origin xyz=0 0.227 0 rpy=1.5707963267949 -1.22460635382238E-16 -3.14159265358979 -> xyz=0 0.227 0 rpy=1.5708 -1.2246E-16 -3.1416; type continuous -> revolute
