Commit message: try again

File: RA605_710/robots/RA605_710.xacro (robot description, xacro)
@@ -1,19 +1,21 @@
+<?xml version="1.0"?>
 <robot
-  name="RA605_710.SLDASM">
+  name="RA605_710" xmlns:xacro="http://www.ros.org/wiki/xacro">
+  <xacro:include filename="$(find RA605_710)/robots/RA605_710.gazebo" />
   <link
     name="base_link">
     <inertial>
       <origin
-        xyz="-0.0032233 -0.005 4.3569E-16"
+        xyz="-0.00322329614662995 -0.005 4.34971473156821E-16"
         rpy="0 0 0" />
       <mass
-        value="39.999" />
+        value="39.9992146018366" />
       <inertia
-        ixx="13.334"
-        ixy="2.1807E-19"
-        ixz="-2.7365E-15"
-        iyy="26.667"
-        iyz="-4.5749E-14"
-        izz="13.334" />
+        ixx="13.3336666552129"
+        ixy="2.18068724778341E-19"
+        ixz="-2.73645750664298E-15"
+        iyy="26.6666666568492"
+        iyz="-4.57489937427496E-14"
+        izz="13.3336666552129" />
     </inertial>
     <visual>
@@ -23,10 +25,10 @@
       <geometry>
         <mesh
-          filename="package://RA605_710.SLDASM/meshes/base_link.STL" />
+          filename="package://RA605_710/meshes/base_link.STL" />
       </geometry>
       <material
         name="">
         <color
-          rgba="0.79216 0.81961 0.93333 1" />
+          rgba="0.792156862745098 0.819607843137255 0.933333333333333 1" />
       </material>
     </visual>
@@ -37,5 +39,5 @@
       <geometry>
         <mesh
-          filename="package://RA605_710.SLDASM/meshes/base_link.STL" />
+          filename="package://RA605_710/meshes/base_link.STL" />
       </geometry>
     </collision>
@@ -45,15 +47,15 @@
     <inertial>
       <origin
-        xyz="-0.0032233 -0.005 3.797E-16"
+        xyz="-0.00322329614662996 -0.005 3.79695301389313E-16"
         rpy="0 0 0" />
       <mass
-        value="39.999" />
+        value="39.9992146018366" />
       <inertia
-        ixx="13.334"
-        ixy="9.0784E-18"
-        ixz="-1.8504E-15"
-        iyy="26.667"
-        iyz="-4.5736E-14"
-        izz="13.334" />
+        ixx="13.3336666552129"
+        ixy="9.07838619093324E-18"
+        ixz="-1.85037170770859E-15"
+        iyy="26.6666666568492"
+        iyz="-4.57355368706325E-14"
+        izz="13.3336666552129" />
     </inertial>
     <visual>
@@ -63,10 +65,10 @@
       <geometry>
         <mesh
-          filename="package://RA605_710.SLDASM/meshes/Link1.STL" />
+          filename="package://RA605_710/meshes/Link1.STL" />
       </geometry>
       <material
         name="">
         <color
-          rgba="0.79216 0.81961 0.93333 1" />
+          rgba="0.792156862745098 0.819607843137255 0.933333333333333 1" />
       </material>
     </visual>
@@ -77,5 +79,5 @@
       <geometry>
         <mesh
-          filename="package://RA605_710.SLDASM/meshes/Link1.STL" />
+          filename="package://RA605_710/meshes/Link1.STL" />
       </geometry>
     </collision>
@@ -116,5 +118,5 @@
       <geometry>
         <mesh
-          filename="package://RA605_710.SLDASM/meshes/Link2.STL" />
+          filename="package://RA605_710/meshes/Link2.STL" />
       </geometry>
       <material
@@ -130,5 +132,5 @@
       <geometry>
         <mesh
-          filename="package://RA605_710.SLDASM/meshes/Link2.STL" />
+          filename="package://RA605_710/meshes/Link2.STL" />
       </geometry>
     </collision>
@@ -147,8 +149,18 @@
       xyz="0 0 1" />
     <limit
+      effort="0"
+      velocity="0"
       lower="-3.1"
-      upper="3.1"
-      effort="0"
-      velocity="0" />
+      upper="3.1" />
   </joint>
+  <transmission name="tran1">
+    <type>transmission_interface/SimpleTransmission</type>
+    <joint name="j2">
+      <hardwareInterface>hardware_interface/EffortJointInterface</hardwareInterface>
+    </joint>
+    <actuator name="motor1">
+      <hardwareInterface>hardware_interface/EffortJointInterface</hardwareInterface>
+      <mechanicalReduction>1</mechanicalReduction>
+    </actuator>
+  </transmission>
 </robot>
