Commit message: fix

File: RA605_710_GB/robots/RA605_710_GB.urdf (robot description, URDF)
Before this commit: robot RA605_710_GB, 9 links, 8 joints
Links:
- link Link6: mass 0.5 -> 1
- link base_Link: mass 50.696 -> 50.6963005253788
- link base_link: mass 1000 -> 39.9992146018366
- link wire: mass 0.21821 -> 0.21821313758791
Joints:
- joint base_fix: origin xyz=0 0 0 rpy=1.5708 0 3.1416 -> xyz=0 0 0 rpy=1.5707963267949 0 3.14159265358979
- joint joint3: origin xyz=0.03322329614663 0 0.148 rpy=0 0 0 -> xyz=0.033223 0 0.148 rpy=0 0 0
- joint joint4: origin xyz=0 0 0.340000000000006 rpy=0 0 0 -> xyz=0 0 0.34 rpy=0 0 0

Commit message: all test

File: RA605_710_GB/robots/RA605_710_GB.urdf (robot description, URDF)
Before this commit: robot RA605_710_GB, 9 links, 8 joints
Links:
- removed link base_link
- removed link wire
- added link base, mass 100; collision mesh filename=package://RA605_710_GB/meshes/base.STL; visual mesh filename=package://RA605_710_GB/meshes/base.STL
- link Link2: mass 50.696 -> 50.478
- link Link4: mass 50.696 -> 50.478
- link Link6: mass 1 -> 2.6849E-06
- link base_Link: mass 50.6963005253788 -> 50.478
Joints:
- removed joint wire
- joint base_fix: origin xyz=0 0 0 rpy=1.5707963267949 0 3.14159265358979 -> xyz=0 0 0 rpy=1.5708 0 3.1416; parent base_link -> base
- joint joint2: origin xyz=0 0.227 0 rpy=1.5707963267949 -1.22460635382238E-16 -3.14159265358979 -> xyz=0 0.227 0 rpy=1.5708 -1.2246E-16 -3.1416
- joint joint3: origin xyz=0.033223 0 0.148 rpy=0 0 0 -> xyz=0.03322329614663 0 0.148 rpy=0 0 0
- joint joint4: origin xyz=0 0 0.34 rpy=0 0 0 -> xyz=0 0 0.340000000000006 rpy=0 0 0
