Commit message: inventor convert

File: ra605/robots/ra605.urdf (robot description, URDF)
Before this commit: robot ra605, 8 links, 7 joints
Links:
- removed link Link1
- removed link floor
- added link Link8, mass 0.10765; collision mesh filename=package://ra605/meshes/Link8.STL; visual mesh filename=package://ra605/meshes/Link8.STL
- added link floor1, mass 39.999; collision mesh filename=package://ra605/meshes/floor1.STL; visual mesh filename=package://ra605/meshes/floor1.STL
- link Link2: mass 50.478 -> 21.943
- link Link3: mass 7.4696 -> 7.6212
- link Link4: mass 50.478 -> 20.11
- link Link5: mass 2.9699 -> 6.7196
- link Link6: mass 2.6849E-06 -> 3.0032
- link Link7: mass 0.039323 -> 1.025
Joints:
- removed joint joint3
- added joint joint8: type continuous, parent Link7, child Link8, origin xyz=0.0677 0 0 rpy=0 0 0, axis 1 0 0
- joint joint1: child Link1 -> Link2; origin xyz=0 0 0 rpy=0 0 0 -> xyz=0 0 0 rpy=0 -1.2246E-16 3.1416; parent floor -> floor1
- joint joint2: child Link2 -> Link3; origin xyz=0 0 0.227 rpy=0 0 0 -> xyz=0.027867 0.1185 0 rpy=1.5708 -1.2246E-16 -3.1416; parent Link1 -> Link2
- joint joint4: origin xyz=0 0 0.34 rpy=0 0 0 -> xyz=0.03 0 0.145 rpy=0 0 0
- joint joint5: axis 1 0 0 -> 0 1 0; origin xyz=0.099 0 0.04 rpy=0 0 0 -> xyz=0 0 0.34 rpy=0 0 0
- joint joint6: axis 0 1 0 -> 1 0 0; origin xyz=0.239 0 0 rpy=0 0 0 -> xyz=0.0989999999999995 0 0.0400000000000098 rpy=0 0 0
- joint joint7: axis 1 0 0 -> 0 1 0; origin xyz=0.0865 0 0 rpy=0 0 0 -> xyz=0.239 0 0 rpy=0 0 0
